File: USB_Hub_ASIC/usb_hub_asic.sch (EAGLE design)
At the start: 1 part, among them U1 IC_CYUSB3314_QUAD_USB3.0_HUB

Commit message: Basic CYUSB3314 connections started
Parts:
- added C1, C2: 10p, rcl:C-USC0805
- added C3, C4: 22u, rcl:C-USC0805
- added C5: 1.5u, rcl:C-USC0805
- added C6, C7, C8, C9: 150u, rcl:CPOL-USSANYO_SMD_E12
- added DS1, DS2, DS3, DS4: CONN_RCPT_USB3.0_TYPEA_9POS_R/A, USB_Hub_ASIC:CONN_RCPT_USB3.0_TYPEA_9POS_R/A
- added FB1, FB2, FB3, FB4: 220Ω, SparkFun-Coils:FERRITE_BEAD-0805-220Ω-100MHZ-2A
- added Q1: 26M, crystal:CRYSTALHC49S
- added R1: 6.04k±1%, rcl:R-US_R0805
- added R2: 200±1%, rcl:R-US_R0805
- added R3, R4, R5: 10k, rcl:R-US_R0805
- added S1: MOMENTARY-SWITCH-SPST-SMD-12MM, SparkFun-Switches:MOMENTARY-SWITCH-SPST-SMD-12MM
Connections:
- new net +1V2: C3.1, U1.AVDD12, U1.DVDD12, U1.VDD_EFUSE
- new net +3V3: C4.1, R3.2, R4.2, R5.2, U1.AVDD33, U1.RESERVED1, U1.VDD_IO
- new net DS1_AMBER/ACA_DOCK: U1.DS1_AMBER/ACA_DOCK
- new net DS1_DM: U1.DS1_DM
- new net DS1_DP: U1.DS1_DP
- new net DS1_GREEN/PORT_DISABLE[0]: U1.DS1_GREEN/PORT_DISABLE[0]
- new net DS1_LED_SS/PORT_DISABLE[1]: U1.DS1_LED_SS/PORT_DISABLE[1]
- new net DS1_OVRCURR: U1.DS1_OVRCURR
- new net DS1_PWREN/CDP_EN: U1.DS1_PWREN/CDP_EN
- new net DS1_RXM: U1.DS1_RXM
- new net DS1_RXP: U1.DS1_RXP
- new net DS1_TXM: U1.DS1_TXM
- new net DS1_TXP: U1.DS1_TXP
- new net DS1_VBUS: FB1.2
- new net DS2_AMBER/NON_REMOVABLE[0]: U1.DS2_AMBER/NON_REMOVABLE[0]
- new net DS2_DM: U1.DS2_DM
- new net DS2_DP: U1.DS2_DP
- new net DS2_GREEN/NON_REMOVABLE[1]: U1.DS2_GREEN/NON_REMOVABLE[1]
- new net DS2_LED_SS/PWR_EN_SEL: U1.DS2_LED_SS/PWR_EN_SEL
- new net DS2_OVRCURR: U1.DS2_OVRCURR
- new net DS2_PWREN/CDP_EN: U1.DS2_PWREN/CDP_EN
- new net DS2_RXM: U1.DS2_RXM
- new net DS2_RXP: U1.DS2_RXP
- new net DS2_TXM: U1.DS2_TXM
- new net DS2_TXP: U1.DS2_TXP
- new net DS2_VBUS: FB2.2
- new net DS3_AMBER/VID_SEL[2]: U1.DS3_AMBER/VID_SEL[2]
- new net DS3_DM: U1.DS3_DM
- new net DS3_DP: U1.DS3_DP
- new net DS3_GREEN/VID_SEL[1]: U1.DS3_GREEN/VID_SEL[1]
- new net DS3_LED_SS/PIN_STRAP: U1.DS3_LED_SS/PIN_STRAP
- new net DS3_OVRCURR: U1.DS3_OVRCURR
- new net DS3_PWREN/CDP_EN: U1.DS3_PWREN/CDP_EN
- new net DS3_RXM: U1.DS3_RXM
- new net DS3_RXP: U1.DS3_RXP
- new net DS3_TXM: U1.DS3_TXM
- new net DS3_TXP: U1.DS3_TXP
- new net DS3_VBUS: FB3.2
- new net DS4_AMBER/I2C_DEV_ID: U1.DS4_AMBER/I2C_DEV_ID
- new net DS4_DM: U1.DS4_DM
- new net DS4_DP: U1.DS4_DP
- new net DS4_GREEN/VID_SEL[0]: U1.DS4_GREEN/VID_SEL[0]
- new net DS4_LED_SS: U1.DS4_LED_SS
- new net DS4_OVRCURR: U1.DS4_OVRCURR
- new net DS4_PWREN/CDP_EN: U1.DS4_PWREN/CDP_EN
- new net DS4_RXM: U1.DS4_RXM
- new net DS4_RXP: U1.DS4_RXP
- new net DS4_TXM: U1.DS4_TXM
- new net DS4_TXP: U1.DS4_TXP
- new net DS4_VBUS: FB4.2
- new net GND: C1.2, C2.2, C3.2, C4.2, C5.2, C6.-, C7.-, C8.-, C9.-, DS1.GND, DS1.GND_DRAIN, DS2.GND, DS2.GND_DRAIN, DS3.GND, DS3.GND_DRAIN, DS4.GND, DS4.GND_DRAIN, R1.1, R2.1, S1.2, U1.GND
- new net I2C_CLK: U1.I2C_CLK
- new net I2C_DATA: U1.I2C_DATA
- new net MODE_SEL[0]: R4.1, U1.MODE_SEL[0]
- new net MODE_SEL[1]: R5.1, U1.MODE_SEL[1]
- new net N$3: C6.+, DS1.VBUS, FB1.1
- new net N$4: C7.+, DS2.VBUS, FB2.1
- new net N$6: C8.+, DS3.VBUS, FB3.1
- new net N$8: C9.+, DS4.VBUS, FB4.1
- new net PWR_SW_POL: U1.PWR_SW_POL
- new net RREF_SS: R2.2, U1.RREF_SS
- new net RREF_USB2: R1.2, U1.RREF_USB2
- new net SUSPEND: U1.SUSPEND
- new net US_DM: U1.US_DM
- new net US_DP: U1.US_DP
- new net US_OVRCURR: U1.US_OVRCURR
- new net US_RXM: U1.US_RXM
- new net US_RXP: U1.US_RXP
- new net US_TXM: U1.US_TXM
- new net US_TXP: U1.US_TXP
- new net VBUS_DS: U1.VBUS_DS
- new net VBUS_US: U1.VBUS_US
- new net XLT_IN: U1.XLT_IN
- new net XTL_IN: C1.1, Q1.1
- new net XTL_OUT: C2.1, Q1.2, U1.XTL_OUT
- new net ~RESETIN: C5.1, R3.1, S1.1, U1.~RESETIN
Other:
- note added: "Configuration mode select (Internal ROM configuration)"
- note added: "Poweron Reset"
- note added: "Precision Calibration Resistors"

Commit message: USB port connections and CYUSB3314 decoupling considerations
Parts:
- removed FB3, FB4: 220Ω, SparkFun-Coils:FERRITE_BEAD-0805-220Ω-100MHZ-2A
- added C10, C11, C12, C13, C14, C15, C16, C17: 0.1u, rcl:C-USC0805
- added C18, C19, C20, C21: 22u, rcl:C-USC0805
- C6, C7, C8, C9: value 150u -> 1u
Connections:
- removed net DS1_VBUS: FB1.2
- removed net DS2_VBUS: FB2.2
- removed net DS3_VBUS: FB3.2
- removed net DS4_VBUS: FB4.2
- removed net N$6: C8.+, DS3.VBUS, FB3.1
- removed net N$8: C9.+, DS4.VBUS, FB4.1
- removed net ~RESETIN: C5.1, R3.1, S1.1, U1.~RESETIN
- new net +5V: C6.+, C7.+, C8.+, C9.+, DS1.VBUS, DS2.VBUS, DS3.VBUS, DS4.VBUS
- new net N$1: C11.2, DS1.SSTXM
- new net N$10: C12.2, DS2.SSTXP
- new net N$13: C15.2, DS3.SSTXM
- new net N$14: C14.2, DS3.SSTXP
- new net N$17: C17.2, DS4.SSTXM
- new net N$18: C16.2, DS4.SSTXP
- new net N$2: C10.2, DS1.SSTXP
- new net N$9: C13.2, DS2.SSTXM
- new net RESETIN: C5.1, R3.1, S1.1, U1.RESETIN
- net +1V2: now also C20.1, C21.1, FB1.1; no longer C3.1, U1.DVDD12
- net +3V3: now also C18.1, C19.1, FB2.1; no longer C4.1, U1.AVDD33
- net DS1_DM: now also DS1.DM
- net DS1_DP: now also DS1.DP
- net DS1_RXM: now also DS1.SSRXM
- net DS1_RXP: now also DS1.SSRXP
- net DS1_TXM: now also C11.1
- net DS1_TXP: now also C10.1
- net DS2_DM: now also DS2.DM
- net DS2_DP: now also DS2.DP
- net DS2_RXM: now also DS2.SSRXM
- net DS2_RXP: now also DS2.SSRXP
- net DS2_TXM: now also C13.1
- net DS2_TXP: now also C12.1
- net DS3_DM: now also DS3.DM
- net DS3_DP: now also DS3.DP
- net DS3_RXM: now also DS3.SSRXM
- net DS3_RXP: now also DS3.SSRXP
- net DS3_TXM: now also C15.1
- net DS3_TXP: now also C14.1
- net DS4_DM: now also DS4.DM
- net DS4_DP: now also DS4.DP
- net DS4_RXM: now also DS4.SSRXM
- net DS4_RXP: now also DS4.SSRXP
- net DS4_TXM: now also C17.1
- net DS4_TXP: now also C16.1
- net GND: now also C18.2, C19.2, C20.2, C21.2, DS1.SHIELD, DS2.SHIELD, DS3.SHIELD, DS4.SHIELD, U1.EPAD
- net N$3: now also C3.1, FB1.2, U1.DVDD12; no longer C6.+, DS1.VBUS, FB1.1
- net N$4: now also C4.1, FB2.2, U1.AVDD33; no longer C7.+, DS2.VBUS, FB2.1

Commit message: Hub configuration straps, LEDs, WIP power
Parts:
- added C22, C24: 0.1u, rcl:C-USC0805
- added C23: 1u, rcl:CPOL-USSANYO_SMD_E12
- added C25, C26: 4.7u, rcl:CPOL-USSANYO_SMD_E12
- added D1, D5: (no value), SparkFun-LED:LED1206
- added D10, D13, D3, D7: GREEN, SparkFun-LED:LED-GREEN1206
- added D11, D14, D4, D8: RED, SparkFun-LED:LED-RED1206
- added D12, D2, D6, D9: BLUE, SparkFun-LED:LED-BLUE1206
- added J5: CONN_RCPT_USB3.0_TYPEB_9POS_R/A, USB_Hub_ASIC:CONN_RCPT_USB3.0_TYPEB_9POS_R/A
- added L1: 4.7u, rcl:L-USCEP125
- added R10, R12, R14, R16, R18, R20, R22, R24, R26, R28, R30, R8: 1k, rcl:R-US_R0805
- added R11, R13, R15, R17, R19, R21, R23, R25, R27, R29, R31, R32, R33, R34, R35, R36, R37, R38, R39, R9: 10k, rcl:R-US_R0805
- added R6, R7: 330, rcl:R-US_R0805
- added U2: IC_MCP1603LT-330_3.3V_500MA_BUCK_REG, USB_Hub_ASIC:IC_MCP1603LT-330_3.3V_500MA_BUCK_REG
- C1: value 10p -> 1.5u
- C12, C13: value 0.1u -> 1u; device rcl:C-USC0805 -> rcl:CPOL-USSANYO_SMD_E12
- C18, C19: value 22u -> 1u; device rcl:C-USC0805 -> rcl:CPOL-USSANYO_SMD_E12
- C2: value 10p -> 22u
- C20, C21: value 22u -> 0.1u
- C5: value 1.5u -> 22u
- C6, C7: value 1u -> 22u; device rcl:CPOL-USSANYO_SMD_E12 -> rcl:C-USC0805
- C8, C9: value 1u -> 10p; device rcl:CPOL-USSANYO_SMD_E12 -> rcl:C-USC0805
- R1: value 6.04k±1% -> 10k
- R3: value 10k -> 6.04k±1%
- renumbered DS1 to J1, DS2 to J3, DS3 to J2, DS4 to J4
Connections:
- removed net VBUS_DS: U1.VBUS_DS
- removed net VBUS_US: U1.VBUS_US
- new net N$11: D4.C, R12.1
- new net N$12: R12.2, R13.2, R18.2, R19.2, R24.2, R25.2, R27.2, R30.2, R31.2, R32.2, R33.2, R34.2, R35.2
- new net N$15: D8.C, R18.1
- new net N$16: D3.C, R10.1
- new net N$19: R10.2, R11.2, R16.2, R17.2, R22.2, R23.2, R28.2, R29.2
- new net N$20: D7.C, R16.1
- new net N$21: D2.C, R8.1
- new net N$22: C26.+, L1.2, R14.2, R15.2, R20.2, R21.2, R36.2, R37.2, R38.2, R39.2, R8.2, R9.2, U2.FB
- new net N$23: D6.C, R14.1
- new net N$24: D9.A, R20.1
- new net N$25: D10.A, R22.1
- new net N$26: D11.A, R24.1
- new net N$27: D14.C, R30.1
- new net N$29: D12.C, R26.1
- new net N$30: L1.1, U2.LX
- new net N$5: C22.2, J5.SSTXM
- new net N$6: C24.2, J5.SSTXP
- new net N$7: D1.C, R6.2
- new net N$8: D5.C, R7.2
- net +1V2: now also C2.1, C3.1; no longer C20.1, C21.1
- net +3V3: now also C4.1, C5.1, R1.2; no longer C18.1, C19.1, R3.2
- net +5V: now also C12.+, C13.+, C18.+, C19.+, C23.+, C25.+, D5.A, J5.VBUS, U1.VBUS_DS, U1.VBUS_US, U2.SHDN, U2.VIN; no longer C6.+, C7.+, C8.+, C9.+
- net DS1_AMBER/ACA_DOCK: now also D4.A, R13.1
- net DS1_GREEN/PORT_DISABLE[0]: now also D3.A, R11.1
- net DS1_LED_SS/PORT_DISABLE[1]: now also D2.A, R9.1
- net DS1_OVRCURR: now also R36.1
- net DS1_PWREN/CDP_EN: now also R27.1
- net DS1_TXM: now also C14.1; no longer C11.1
- net DS2_AMBER/NON_REMOVABLE[0]: now also D8.A, R19.1
- net DS2_GREEN/NON_REMOVABLE[1]: now also D7.A, R17.1
- net DS2_LED_SS/PWR_EN_SEL: now also D6.A, R15.1
- net DS2_OVRCURR: now also R37.1
- net DS2_PWREN/CDP_EN: now also R33.1
- net DS2_TXM: now also C20.1; no longer C13.1
- net DS2_TXP: now also C16.1; no longer C12.1
- net DS3_AMBER/VID_SEL[2]: now also D11.C, R25.1
- net DS3_GREEN/VID_SEL[1]: now also D10.C, R23.1
- net DS3_LED_SS/PIN_STRAP: now also D9.C, R21.1
- net DS3_OVRCURR: now also R38.1
- net DS3_PWREN/CDP_EN: now also R34.1
- net DS3_TXP: now also C11.1; no longer C14.1
- net DS4_AMBER/I2C_DEV_ID: now also D14.A, R31.1
- net DS4_GREEN/VID_SEL[0]: now also D13.A, D13.C, R28.1, R29.1
- net DS4_LED_SS: now also D12.A
- net DS4_OVRCURR: now also R39.1
- net DS4_PWREN/CDP_EN: now also R35.1
- net DS4_TXM: now also C21.1; no longer C17.1
- net DS4_TXP: now also C17.1; no longer C16.1
- net GND: now also C12.-, C13.-, C18.-, C19.-, C23.-, C25.-, C26.-, C6.2, C7.2, C8.2, C9.2, J5.GND, J5.GND_DRAIN, J5.SHIELD, R26.2, R3.1, R6.1, R7.1, U2.GND; no longer C18.2, C19.2, C20.2, C21.2, C6.-, C7.-, C8.-, C9.-, R1.1
- net N$1: now also C14.2; no longer C11.2
- net N$10: now also C16.2; no longer C12.2
- net N$14: now also C11.2; no longer C14.2
- net N$17: now also C21.2; no longer C17.2
- net N$18: now also C17.2; no longer C16.2
- net N$3: now also C7.1; no longer C3.1
- net N$4: now also C6.1; no longer C4.1
- net N$9: now also C20.2; no longer C13.2
- net PWR_SW_POL: now also R32.1
- net RESETIN: now also C1.1, R1.1; no longer C5.1, R3.1
- net RREF_USB2: now also R3.2; no longer R1.2
- net SUSPEND: now also D1.A
- net US_DM: now also J5.DM
- net US_DP: now also J5.DP
- net US_RXM: now also J5.SSRXM
- net US_RXP: now also J5.SSRXP
- net US_TXM: now also C22.1
- net US_TXP: now also C24.1
- net XTL_IN: now also C8.1; no longer C1.1
- net XTL_OUT: now also C9.1; no longer C2.1
Other:
- note added: "Crystal Oscillator"
- note added: "Pin Strap configuration & Blinkenlights"
- moved on the sheet: C1, C11, C14, C16, C17, C2, C20, C21, C3, C4, C5, Q1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

Commit message: Preliminary Design Review Pre-Baseline
Parts:
- removed C14, C16: 0.1u, rcl:C-USC0805
- added C27: 150u, rcl:CPOL-USSANYO_SMD_E12
- added C28, C29, C30, C31, C32, C33, C34: 0.1u, rcl:C-USC0805
- added FB3, FB4, FB5, FB6: 220Ω, SparkFun-Coils:FERRITE_BEAD-0805-220Ω-100MHZ-2A
- added L2: 2.2u, rcl:L-USCEP125
- added R40, R46, R47: 10k, rcl:R-US_R0805
- added R41, R42, R43, R44, R45: 1M, rcl:R-US_R0805
- added U3: IC_LM3674MF-1.2/NOPB_1.2V_600MA_BUCK_REG, USB_Hub_ASIC:IC_LM3674MF-1.2/NOPB_1.2V_600MA_BUCK_REG
- C1: value 1.5u -> 4.7u; device rcl:C-USC0805 -> rcl:CPOL-USSANYO_SMD_E12
- C10, C11: value 0.1u -> 22u
- C12, C13: value 1u -> 10p; device rcl:CPOL-USSANYO_SMD_E12 -> rcl:C-USC0805
- C18, C19, C23: value 1u -> 0.1u; device rcl:CPOL-USSANYO_SMD_E12 -> rcl:C-USC0805
- C2: value 22u -> 1.5u
- C20: value 0.1u -> 150; device rcl:C-USC0805 -> rcl:CPOL-USSANYO_SMD_E12
- C21: value 0.1u -> 150u; device rcl:C-USC0805 -> rcl:CPOL-USSANYO_SMD_E12
- C25: value 4.7u -> 0.1u; device rcl:CPOL-USSANYO_SMD_E12 -> rcl:C-USC0805
- C26: value 4.7u -> 150u
- C3, C4: value 22u -> 4.7u; device rcl:C-USC0805 -> rcl:CPOL-USSANYO_SMD_E12
- C5: value 22u -> 10u; device rcl:C-USC0805 -> rcl:CPOL-USSANYO_SMD_E12
- C8, C9: value 10p -> 22u
- D10, D13, D7: value GREEN -> BLUE; device SparkFun-LED:LED-GREEN1206 -> SparkFun-LED:LED-BLUE1206
- D11: value RED -> GREEN; device SparkFun-LED:LED-RED1206 -> SparkFun-LED:LED-GREEN1206
- D12, D2: value BLUE -> RED; device SparkFun-LED:LED-BLUE1206 -> SparkFun-LED:LED-RED1206
- D14: value RED -> (none); device SparkFun-LED:LED-RED1206 -> SparkFun-LED:LED1206
- D4: value RED -> BLUE; device SparkFun-LED:LED-RED1206 -> SparkFun-LED:LED-BLUE1206
- D5: value (none) -> RED; device SparkFun-LED:LED1206 -> SparkFun-LED:LED-RED1206
- D6, D9: value BLUE -> GREEN; device SparkFun-LED:LED-BLUE1206 -> SparkFun-LED:LED-GREEN1206
- J1: value CONN_RCPT_USB3.0_TYPEA_9POS_R/A -> CONN_RCPT_USB3.0_TYPEB_9POS_R/A; device USB_Hub_ASIC:CONN_RCPT_USB3.0_TYPEA_9POS_R/A -> USB_Hub_ASIC:CONN_RCPT_USB3.0_TYPEB_9POS_R/A
- J5: value CONN_RCPT_USB3.0_TYPEB_9POS_R/A -> CONN_RCPT_USB3.0_TYPEA_9POS_R/A; device USB_Hub_ASIC:CONN_RCPT_USB3.0_TYPEB_9POS_R/A -> USB_Hub_ASIC:CONN_RCPT_USB3.0_TYPEA_9POS_R/A
- R11, R13, R17, R19, R27, R9: value 10k -> 1k
- R15: value 10k -> 200±1%
- R16: value 1k -> 6.04k±1%
- R2: value 200±1% -> 330
- R22, R24, R26, R30, R8: value 1k -> 10k
- R3: value 6.04k±1% -> 10k
- R36: value 10k -> 330
- R6, R7: value 330 -> 10k
- U1: value IC_CYUSB3314_QUAD_USB3.0_HUB -> IC_MCP1603LT-330_3.3V_500MA_BUCK_REG; device USB_Hub_ASIC:IC_CYUSB3314_QUAD_USB3.0_HUB -> USB_Hub_ASIC:IC_MCP1603LT-330_3.3V_500MA_BUCK_REG
- U2: value IC_MCP1603LT-330_3.3V_500MA_BUCK_REG -> IC_CYUSB3314_QUAD_USB3.0_HUB; device USB_Hub_ASIC:IC_MCP1603LT-330_3.3V_500MA_BUCK_REG -> USB_Hub_ASIC:IC_CYUSB3314_QUAD_USB3.0_HUB
Connections:
- removed net N$19: R10.2, R11.2, R16.2, R17.2, R22.2, R23.2, R28.2, R29.2
- removed net N$22: C26.+, L1.2, R14.2, R15.2, R20.2, R21.2, R36.2, R37.2, R38.2, R39.2, R8.2, R9.2, U2.FB
- new net N$28: L2.1, U3.SW
- new net N$31: C10.1, C11.1, FB1.2, U2.DVDD12, U2.VDD_EFUSE
- new net N$32: D11.A, R20.1
- new net N$33: FB5.2, J4.VBUS
- new net N$34: FB4.2, J3.VBUS
- new net N$35: FB6.2, J5.VBUS
- new net N$36: R46.1, R47.1, U2.VBUS_US
- new net N$37: C30.1, J1.SHIELD, R41.2
- new net N$38: C31.1, J2.SHIELD, R42.2
- new net N$39: C32.1, J4.SHIELD, R43.2
- new net N$40: C33.1, J3.SHIELD, R44.2
- new net N$41: C34.1, J5.SHIELD, R45.2
- new net VBUS_US: J1.VBUS, R46.2
- net +1V2: now also C5.+, C6.1, L2.2, U2.AVDD12, U3.FB; no longer C2.1, C3.1, U1.AVDD12, U1.VDD_EFUSE
- net +3V3: now also C3.+, C7.1, C8.1, L1.2, R17.2, R18.2, R19.2, R20.2, R21.2, R22.2, R23.2, R24.2, R25.2, R29.2, R30.2, R37.2, R38.2, R39.2, R40.2, U1.FB, U2.RESERVED1, U2.VDD_IO; no longer C4.1, C5.1, R4.2, R5.2, U1.RESERVED1, U1.VDD_IO
- net +5V: now also C1.+, C20.+, C21.+, C26.+, C27.+, C4.+, D14.A, FB3.1, FB4.1, FB5.1, FB6.1, U1.SHDN, U1.VIN, U2.VBUS_DS, U3.EN, U3.VIN; no longer C12.+, C13.+, C18.+, C19.+, C23.+, C25.+, D5.A, J1.VBUS, J2.VBUS, J3.VBUS, J4.VBUS, J5.VBUS, U1.VBUS_DS, U1.VBUS_US, U2.SHDN, U2.VIN
- net DS1_AMBER/ACA_DOCK: now also D2.A, R3.1, U2.DS1_AMBER/ACA_DOCK; no longer D4.A, R13.1, U1.DS1_AMBER/ACA_DOCK
- net DS1_DM: now also J2.DM, U2.DS1_DM; no longer J1.DM, U1.DS1_DM
- net DS1_DP: now also J2.DP, U2.DS1_DP; no longer J1.DP, U1.DS1_DP
- net DS1_GREEN/PORT_DISABLE[0]: now also R4.1, U2.DS1_GREEN/PORT_DISABLE[0]; no longer R11.1, U1.DS1_GREEN/PORT_DISABLE[0]
- net DS1_LED_SS/PORT_DISABLE[1]: now also D4.A, R5.1, U2.DS1_LED_SS/PORT_DISABLE[1]; no longer D2.A, R9.1, U1.DS1_LED_SS/PORT_DISABLE[1]
- net DS1_OVRCURR: now also R37.1, U2.DS1_OVRCURR; no longer R36.1, U1.DS1_OVRCURR
- net DS1_PWREN/CDP_EN: now also R32.1, U2.DS1_PWREN/CDP_EN; no longer R27.1, U1.DS1_PWREN/CDP_EN
- net DS1_RXM: now also J2.SSRXM, U2.DS1_RXM; no longer J1.SSRXM, U1.DS1_RXM
- net DS1_RXP: now also J2.SSRXP, U2.DS1_RXP; no longer J1.SSRXP, U1.DS1_RXP
- net DS1_TXM: now also C22.1, U2.DS1_TXM; no longer C14.1, U1.DS1_TXM
- net DS1_TXP: now also C18.1, U2.DS1_TXP; no longer C10.1, U1.DS1_TXP
- net DS2_AMBER/NON_REMOVABLE[0]: now also D5.A, R6.1, U2.DS2_AMBER/NON_REMOVABLE[0]; no longer D8.A, R19.1, U1.DS2_AMBER/NON_REMOVABLE[0]
- net DS2_DM: now also J4.DM, U2.DS2_DM; no longer J3.DM, U1.DS2_DM
- net DS2_DP: now also J4.DP, U2.DS2_DP; no longer J3.DP, U1.DS2_DP
- net DS2_GREEN/NON_REMOVABLE[1]: now also D6.A, R7.1, U2.DS2_GREEN/NON_REMOVABLE[1]; no longer D7.A, R17.1, U1.DS2_GREEN/NON_REMOVABLE[1]
- net DS2_LED_SS/PWR_EN_SEL: now also D7.A, R8.1, U2.DS2_LED_SS/PWR_EN_SEL; no longer D6.A, R15.1, U1.DS2_LED_SS/PWR_EN_SEL
- net DS2_OVRCURR: now also R38.1, U2.DS2_OVRCURR; no longer R37.1, U1.DS2_OVRCURR
- net DS2_PWREN/CDP_EN: now also U2.DS2_PWREN/CDP_EN; no longer U1.DS2_PWREN/CDP_EN
- net DS2_RXM: now also J4.SSRXM, U2.DS2_RXM; no longer J3.SSRXM, U1.DS2_RXM
- net DS2_RXP: now also J4.SSRXP, U2.DS2_RXP; no longer J3.SSRXP, U1.DS2_RXP
- net DS2_TXM: now also C28.1, U2.DS2_TXM; no longer C20.1, U1.DS2_TXM
- net DS2_TXP: now also C24.1, U2.DS2_TXP; no longer C16.1, U1.DS2_TXP
- net DS3_AMBER/VID_SEL[2]: now also D8.C, R22.1, U2.DS3_AMBER/VID_SEL[2]; no longer D11.C, R25.1, U1.DS3_AMBER/VID_SEL[2]
- net DS3_DM: now also J3.DM, U2.DS3_DM; no longer J2.DM, U1.DS3_DM
- net DS3_DP: now also J3.DP, U2.DS3_DP; no longer J2.DP, U1.DS3_DP
- net DS3_GREEN/VID_SEL[1]: now also D9.C, U2.DS3_GREEN/VID_SEL[1]; no longer D10.C, U1.DS3_GREEN/VID_SEL[1]
- net DS3_LED_SS/PIN_STRAP: now also D10.C, R24.1, U2.DS3_LED_SS/PIN_STRAP; no longer D9.C, R21.1, U1.DS3_LED_SS/PIN_STRAP
- net DS3_OVRCURR: now also R39.1, U2.DS3_OVRCURR; no longer R38.1, U1.DS3_OVRCURR
- net DS3_PWREN/CDP_EN: now also U2.DS3_PWREN/CDP_EN; no longer U1.DS3_PWREN/CDP_EN
- net DS3_RXM: now also J3.SSRXM, U2.DS3_RXM; no longer J2.SSRXM, U1.DS3_RXM
- net DS3_RXP: now also J3.SSRXP, U2.DS3_RXP; no longer J2.SSRXP, U1.DS3_RXP
- net DS3_TXM: now also C23.1, U2.DS3_TXM; no longer C15.1, U1.DS3_TXM
- net DS3_TXP: now also C19.1, U2.DS3_TXP; no longer C11.1, U1.DS3_TXP
- net DS4_AMBER/I2C_DEV_ID: now also D12.A, R26.1, U2.DS4_AMBER/I2C_DEV_ID; no longer D14.A, R31.1, U1.DS4_AMBER/I2C_DEV_ID
- net DS4_DM: now also J5.DM, U2.DS4_DM; no longer J4.DM, U1.DS4_DM
- net DS4_DP: now also J5.DP, U2.DS4_DP; no longer J4.DP, U1.DS4_DP
- net DS4_GREEN/VID_SEL[0]: now also D11.C, R25.1, U2.DS4_GREEN/VID_SEL[0]; no longer D13.A, D13.C, R28.1, R29.1, U1.DS4_GREEN/VID_SEL[0]
- net DS4_LED_SS: now also D13.A, U2.DS4_LED_SS; no longer D12.A, U1.DS4_LED_SS
- net DS4_OVRCURR: now also R40.1, U2.DS4_OVRCURR; no longer R39.1, U1.DS4_OVRCURR
- net DS4_PWREN/CDP_EN: now also U2.DS4_PWREN/CDP_EN; no longer U1.DS4_PWREN/CDP_EN
- net DS4_RXM: now also J5.SSRXM, U2.DS4_RXM; no longer J4.SSRXM, U1.DS4_RXM
- net DS4_RXP: now also J5.SSRXP, U2.DS4_RXP; no longer J4.SSRXP, U1.DS4_RXP
- net DS4_TXM: now also C29.1, U2.DS4_TXM; no longer C21.1, U1.DS4_TXM
- net DS4_TXP: now also C25.1, U2.DS4_TXP; no longer C17.1, U1.DS4_TXP
- net GND: now also C1.-, C10.2, C11.2, C12.2, C13.2, C20.-, C21.-, C27.-, C3.-, C30.2, C31.2, C32.2, C33.2, C34.2, C4.-, C5.-, R10.2, R11.2, R12.2, R13.2, R14.2, R15.1, R16.1, R27.2, R28.2, R3.2, R32.2, R33.2, R34.2, R35.2, R36.1, R4.2, R41.1, R42.1, R43.1, R44.1, R45.1, R47.2, R5.2, R6.2, R7.2, R8.2, R9.2, U2.EPAD, U3.GND; no longer C1.2, C12.-, C13.-, C18.-, C19.-, C23.-, C25.-, C3.2, C4.2, C5.2, J1.SHIELD, J2.SHIELD, J3.SHIELD, J4.SHIELD, J5.SHIELD, R3.1, R6.1, R7.1, U1.EPAD
- net I2C_CLK: now also U2.I2C_CLK; no longer U1.I2C_CLK
- net I2C_DATA: now also U2.I2C_DATA; no longer U1.I2C_DATA
- net MODE_SEL[0]: now also R29.1, U2.MODE_SEL[0]; no longer R4.1, U1.MODE_SEL[0]
- net MODE_SEL[1]: now also R30.1, U2.MODE_SEL[1]; no longer R5.1, U1.MODE_SEL[1]
- net N$1: now also C22.2, J2.SSTXM; no longer C14.2, J1.SSTXM
- net N$10: now also C24.2, J4.SSTXP; no longer C16.2, J3.SSTXP
- net N$11: now also D2.C, R9.1; no longer D4.C, R12.1
- net N$12: no longer R12.2, R13.2, R18.2, R19.2, R24.2, R25.2, R27.2, R30.2, R32.2, R33.2, R34.2, R35.2
- net N$13: now also C23.2, J3.SSTXM; no longer C15.2, J2.SSTXM
- net N$14: now also C19.2, J3.SSTXP; no longer C11.2, J2.SSTXP
- net N$15: now also D5.C, R12.1; no longer D8.C, R18.1
- net N$17: now also C29.2, J5.SSTXM; no longer C21.2, J4.SSTXM
- net N$18: now also C25.2, J5.SSTXP; no longer C17.2, J4.SSTXP
- net N$2: now also C18.2, J2.SSTXP; no longer C10.2, J1.SSTXP
- net N$20: now also D6.C, R13.1; no longer D7.C, R16.1
- net N$21: now also D4.C, R11.1; no longer D2.C, R8.1
- net N$23: now also D7.C; no longer D6.C
- net N$24: now also D10.A, R19.1; no longer D9.A, R20.1
- net N$25: now also D9.A, R18.1; no longer D10.A, R22.1
- net N$26: now also D8.A, R17.1; no longer D11.A, R24.1
- net N$27: now also D12.C, R27.1; no longer D14.C, R30.1
- net N$29: now also D13.C, R28.1; no longer D12.C, R26.1
- net N$3: now also FB3.2, J2.VBUS; no longer C7.1, FB1.2, U1.DVDD12
- net N$30: now also U1.LX; no longer U2.LX
- net N$4: now also C9.1, U2.AVDD33; no longer C6.1, U1.AVDD33
- net N$5: now also C15.2, J1.SSTXM; no longer C22.2, J5.SSTXM
- net N$6: now also C17.2, J1.SSTXP; no longer C24.2, J5.SSTXP
- net N$7: now also R2.2; no longer R6.2
- net N$8: now also D14.C, R36.2; no longer D5.C, R7.2
- net N$9: now also C28.2, J4.SSTXM; no longer C20.2, J3.SSTXM
- net PWR_SW_POL: now also R31.1, U2.PWR_SW_POL; no longer R32.1, U1.PWR_SW_POL
- net RESETIN: now also C2.1, U2.RESETIN; no longer C1.1, U1.RESETIN
- net RREF_SS: now also R15.2, U2.RREF_SS; no longer R2.2, U1.RREF_SS
- net RREF_USB2: now also R16.2, U2.RREF_USB2; no longer R3.2, U1.RREF_USB2
- net SUSPEND: now also U2.SUSPEND; no longer U1.SUSPEND
- net US_DM: now also J1.DM, U2.US_DM; no longer J5.DM, U1.US_DM
- net US_DP: now also J1.DP, U2.US_DP; no longer J5.DP, U1.US_DP
- net US_OVRCURR: now also R21.1, U2.US_OVRCURR; no longer U1.US_OVRCURR
- net US_RXM: now also J1.SSRXM, U2.US_RXM; no longer J5.SSRXM, U1.US_RXM
- net US_RXP: now also J1.SSRXP, U2.US_RXP; no longer J5.SSRXP, U1.US_RXP
- net US_TXM: now also C15.1, U2.US_TXM; no longer C22.1, U1.US_TXM
- net US_TXP: now also C17.1, U2.US_TXP; no longer C24.1, U1.US_TXP
- net XLT_IN: now also U2.XLT_IN; no longer U1.XLT_IN
- net XTL_IN: now also C13.1; no longer C8.1
- net XTL_OUT: now also C12.1, U2.XTL_OUT; no longer C9.1, U1.XTL_OUT
Other:
- note added: "Board Power"
- note added: "TODO: 5V Power Jack"
- moved on the sheet: C10, C11, C15, C17, C2, C22, C24, C26, C6, C7, C8, C9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

Commit message: Post design review warning approval
Connections:
- removed net N$12: R31.2
- removed net XLT_IN: U2.XLT_IN
- net GND: now also R31.2
- net XTL_IN: now also U2.XTL_IN
Changed lines of the file:
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@@
 <setting verticaltext="up"/>
 </settings>
-<grid distance="0.1" unitdist="inch" unit="inch" style="lines" multiple="1" display="yes" altdistance="0.01" altunitdist="inch" altunit="inch"/>
+<grid distance="0.1" unitdist="inch" unit="inch" style="lines" multiple="1" display="no" altdistance="0.01" altunitdist="inch" altunit="inch"/>
 <layers>
 <layer number="1" name="Top" color="4" fill="1" visible="no" active="no"/>
@@
 <part name="GND46" library="supply1" library_urn="urn:adsk.eagle:library:371" deviceset="GND" device=""/>
 <part name="GND47" library="supply1" library_urn="urn:adsk.eagle:library:371" deviceset="GND" device=""/>
+<part name="GND48" library="supply1" library_urn="urn:adsk.eagle:library:371" deviceset="GND" device=""/>
 </parts>
 <sheets>
@@
 <attribute name="VALUE" x="231.14" y="307.34" size="1.778" layer="96"/>
 </instance>
+<instance part="GND48" gate="1" x="203.2" y="284.48" smashed="yes">
+<attribute name="VALUE" x="200.66" y="281.94" size="1.778" layer="96"/>
+</instance>
 </instances>
 <busses>
@@
 <junction x="160.02" y="157.48"/>
 <label x="147.32" y="157.48" size="1.778" layer="95"/>
-</segment>
-</net>
-<net name="XLT_IN" class="0">
-<segment>
-<pinref part="U2" gate="G$1" pin="XLT_IN"/>
-<wire x1="137.16" y1="99.06" x2="157.48" y2="99.06" width="0.1524" layer="91"/>
-<label x="154.94" y="99.06" size="1.778" layer="95" align="bottom-right"/>
 </segment>
 </net>
@@
 <pinref part="GND47" gate="1" pin="GND"/>
 </segment>
+<segment>
+<pinref part="R31" gate="G$1" pin="2"/>
+<wire x1="195.58" y1="289.56" x2="203.2" y2="289.56" width="0.1524" layer="91"/>
+<wire x1="203.2" y1="289.56" x2="203.2" y2="287.02" width="0.1524" layer="91"/>
+<pinref part="GND48" gate="1" pin="GND"/>
+</segment>
 </net>
 <net name="RREF_USB2" class="0">
@@
 <junction x="160.02" y="147.32"/>
 <label x="147.32" y="147.32" size="1.778" layer="95"/>
+</segment>
+<segment>
+<pinref part="U2" gate="G$1" pin="XTL_IN"/>
+<wire x1="137.16" y1="99.06" x2="157.48" y2="99.06" width="0.1524" layer="91"/>
+<label x="154.94" y="99.06" size="1.778" layer="95" align="bottom-right"/>
 </segment>
 </net>
@@
 <pinref part="R9" gate="G$1" pin="1"/>
 <wire x1="58.42" y1="289.56" x2="60.96" y2="289.56" width="0.1524" layer="91"/>
-</segment>
-</net>
-<net name="N$12" class="0">
-<segment>
-<pinref part="R31" gate="G$1" pin="2"/>
-<wire x1="195.58" y1="289.56" x2="203.2" y2="289.56" width="0.1524" layer="91"/>
-<wire x1="203.2" y1="289.56" x2="203.2" y2="287.02" width="0.1524" layer="91"/>
 </segment>
 </net>
@@
 </sheet>
 </sheets>
+<errors>
+</errors>
 </schematic>
 </drawing>

Commit message: moving forward with pcb design
Parts:
- removed C26, C27: 150u, rcl:CPOL-USSANYO_SMD_E12
- removed FB1, FB2, FB3, FB4, FB5, FB6: 220Ω, SparkFun-Coils:FERRITE_BEAD-0805-220Ω-100MHZ-2A
- added C14, C16: 150u, rcl:CPOL-USSANYO_SMD_E12
- C10, C11, C12, C13, C2, C6, C7, C8, C9: device rcl:C-USC0805 -> SparkFun-Capacitors:CAP-0603
- C20: value 150 -> 150u
- D1: value (none) -> SUSPEND
- D10: value BLUE -> DS3_BLU
- D11: value GREEN -> DS4_GRN
- D12: value RED -> DS4_AMB
- D13: value BLUE -> DS4_BLU
- D14: value (none) -> PWR
- D2: value RED -> DS1_AMB
- D3: value GREEN -> DS1_GRN
- D4: value BLUE -> DS1_BLU
- D5: value RED -> DS2_AMB
- D6: value GREEN -> DS2_GRN
- D7: value BLUE -> DS2_BLU
- D8: value RED -> DS3_AMB
- D9: value GREEN -> DS3_GRN
- R1, R10, R11, R12, R13, R14, R15, R16, R17, R18, R19, R2, R20, R21, R22, R23, R24, R25, R26, R27, R28, R29, R3, R30, R31, R32, R33, R34, R35, R36, R37, R38, R39, R4, R40, R41, R42, R43, R44, R45, R46, R47, R5, R6, R7, R8, R9: device rcl:R-US_R0805 -> rcl:R-US_R0603
Connections:
- removed net N$31: C10.1, C11.1, FB1.2, U2.DVDD12, U2.VDD_EFUSE
- removed net N$33: FB5.2, J4.VBUS
- removed net N$34: FB4.2, J3.VBUS
- removed net N$35: FB6.2, J5.VBUS
- removed net N$4: C9.1, FB2.2, U2.AVDD33
- removed net VBUS_US: J1.VBUS, R46.2
- net +1V2: now also C10.1, C11.1, C9.1, U2.DVDD12, U2.VDD_EFUSE; no longer C6.1, FB1.1
- net +3V3: now also C6.1, U2.AVDD33; no longer FB2.1
- net +5V: now also J1.VBUS, R46.2; no longer C20.+, C21.+, C26.+, C27.+, FB3.1, FB4.1, FB5.1, FB6.1
- net GND: now also C14.-, C16.-; no longer C26.-, C27.-
- net N$3: now also C14.+, C16.+, C20.+, C21.+, J3.VBUS, J4.VBUS, J5.VBUS; no longer FB3.2
Other:
- moved on the sheet: C10, C11, C20, C21, C6, C7, C8, C9, D14, R36
