File: USB_Hub_ASIC/usb_hub_asic.brd (EAGLE design)
At the start: 96.5 x 50.8 mm, 105 parts, among them Q1 26M, SW1 RESET, U1 IC_MCP1603LT-330_3.3V_500MA_B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, U2 IC_CYUSB3314_QUAD_USB3.0_HUB, U3 IC_LM3674MF-1.2/NOPB_1.2V_600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

Commit message: start over on board design w/ 4 layers
Parts:
- C2: device SparkFun-Capacitors:0603 -> rcl:C0603
- moved R47 267.7 mm to (-97.8, 104.1)
- moved R46 262.1 mm to (-92.7, 104.1)
- moved R8 260.7 mm to (-82.5, 109.2)
- moved R30 260.6 mm to (-97.8, 99.1)
- moved R7 254.3 mm to (-77.5, 109.2)
- moved R29 253.8 mm to (-92.7, 99.1)
- moved R6 248.4 mm to (-72.4, 109.2)
- moved R4 242.5 mm to (-62.2, 109.2)
- moved R5 242.5 mm to (-67.3, 109.2)
- moved R22 238.0 mm to (-57.1, 99.1)
- moved R3 236.9 mm to (-57.1, 109.2)
- moved R26 235.9 mm to (-77.5, 99.1)
- moved R38 228.9 mm to (-52.1, 104.1)
- moved R16 221.0 mm to (-55.9, 86.4), turned to 0 degrees
- moved R34 215.5 mm to (-31.8, 104.1)
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Routing:
- net DS3_AMBER/VID_SEL[2]: track 84.3 -> 0.00 mm, vias 4 -> 0
- net DS2_AMBER/NON_REMOVABLE[0]: track 80.7 -> 0.00 mm, vias 2 -> 0
- net DS2_GREEN/NON_REMOVABLE[1]: track 78.8 -> 0.00 mm, vias 2 -> 0
- net DS4_LED_SS: track 73.6 -> 0.00 mm
- net DS3_LED_SS/PIN_STRAP: track 72.8 -> 0.00 mm, vias 4 -> 0
- net DS3_GREEN/VID_SEL[1]: track 68.5 -> 0.00 mm, vias 6 -> 0
- net DS4_AMBER/I2C_DEV_ID: track 62.5 -> 0.00 mm
- net +3V3: track 71.9 -> 13.5 mm, vias 9 -> 8
- net DS2_LED_SS/PWR_EN_SEL: track 57.3 -> 0.00 mm, vias 4 -> 0
- net DS3_D_P: track 51.8 -> 0.00 mm, vias 1 -> 0
- net DS3_D_N: track 51.2 -> 0.00 mm, vias 1 -> 0
- net DS4_GREEN/VID_SEL[0]: track 50.9 -> 0.00 mm
- net DS1_LED_SS/PORT_DISABLE[1]: track 47.9 -> 0.00 mm, vias 2 -> 0
- net DS1_D_P: track 47.7 -> 0.00 mm, vias 1 -> 0
- net DS4_D_P: track 47.6 -> 0.00 mm, vias 1 -> 0
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- added copper zone on layer 2, net +1V2
- added copper zone on layer 15, net +3V3
- added copper zone on layer 15, net GND
- added copper zone on layer 2, net GND
- removed copper zone on layer 16, net +1V2
- removed copper zone on layer 16, net +3V3
- removed copper zone on layer 16, net +5V
Other:
- board size 96.5 x 50.8 mm -> 101.6 x 50.8 mm

Commit message: routing is hard
Parts:
- moved R28 208.5 mm to (97.8, 3.81), flipped to the bottom
- moved R27 200.5 mm to (97.8, 11.4), flipped to the bottom
- moved R20 171.2 mm to (97.8, 7.62), flipped to the bottom
- moved C13 163.9 mm to (63.5, 44.5), flipped to the bottom, turned to 90 degrees
- moved R19 156.7 mm to (82.5, 3.81), flipped to the bottom, turned to 90 degrees
- moved R9 156.4 mm to (29.2, 3.81), flipped to the bottom, turned to 90 degrees
- moved R18 155.8 mm to (86.4, 3.81), flipped to the bottom, turned to 90 degrees
- moved Q1 155.0 mm to (59.7, 44.5), flipped to the bottom
- moved R17 154.7 mm to (90.2, 3.81), flipped to the bottom, turned to 90 degrees
- moved R10 152.7 mm to (25.4, 3.81), flipped to the bottom, turned to 90 degrees
- moved C12 151.8 mm to (55.9, 44.5), flipped to the bottom, turned to 270 degrees
- moved R14 123.6 mm to (52.1, 3.81), flipped to the bottom, turned to 90 degrees
- moved R13 122.8 mm to (55.9, 3.81), flipped to the bottom, turned to 90 degrees
- moved R12 122.0 mm to (59.7, 3.81), flipped to the bottom, turned to 90 degrees
- moved R11 113.9 mm to (21.6, 3.81), flipped to the bottom, turned to 90 degrees
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Routing:
- net DS1_LED_SS/PORT_DISABLE[1]: track 0.00 -> 99.1 mm, vias 0 -> 1
- net DS1_GREEN/PORT_DISABLE[0]: track 0.00 -> 95.9 mm, vias 0 -> 1
- net DS1_AMBER/ACA_DOCK: track 0.00 -> 92.7 mm, vias 0 -> 1
- net DS1_D_P: track 0.00 -> 90.4 mm, vias 0 -> 1
- net DS1_D_N: track 0.00 -> 89.7 mm, vias 0 -> 1
- net RESETIN: track 0.00 -> 72.4 mm, vias 0 -> 1
- net DS2_LED_SS/PWR_EN_SEL: track 0.00 -> 63.7 mm, vias 0 -> 1
- net DS3_GREEN/VID_SEL[1]: track 0.00 -> 61.3 mm, vias 0 -> 1
- net DS3_LED_SS/PIN_STRAP: track 0.00 -> 59.7 mm, vias 0 -> 1
- net DS2_GREEN/NON_REMOVABLE[1]: track 0.00 -> 58.9 mm, vias 0 -> 1
- net DS2_D_N: track 0.00 -> 58.6 mm, vias 0 -> 1
- net DS2_AMBER/NON_REMOVABLE[0]: track 0.00 -> 58.2 mm, vias 0 -> 1
- net DS2_D_P: track 0.00 -> 57.8 mm, vias 0 -> 1
- net DS3_D_P: track 0.00 -> 52.8 mm, vias 0 -> 1
- net DS3_AMBER/VID_SEL[2]: track 0.00 -> 52.2 mm, vias 0 -> 1
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
Commit message: ROUTING IS DONE?
Parts:
- moved R45 200.6 mm to (94.0, 19.1), flipped to the bottom, turned to 90 degrees
- moved C34 188.3 mm to (95.2, 19.1), flipped to the bottom, turned to 270 degrees
- moved R44 184.6 mm to (72.4, 3.81), flipped to the bottom, turned to 180 degrees
- moved R41 175.5 mm to (95.2, 38.1), flipped to the bottom, turned to 90 degrees
- moved D1 173.9 mm to (66.0, 35.6)
- moved R47 173.1 mm to (62.2, 38.1), flipped to the bottom, turned to 270 degrees
- moved C33 171.2 mm to (72.4, 2.54), flipped to the bottom
- moved R26 170.4 mm to (73.7, 20.3), turned to 180 degrees
- moved R46 167.0 mm to (62.2, 41.9), flipped to the bottom, turned to 90 degrees
- moved D14 166.4 mm to (78.7, 41.9), turned to 270 degrees
- moved C30 161.1 mm to (94.0, 38.1), flipped to the bottom, turned to 270 degrees
- moved R43 158.9 mm to (45.7, 3.81), flipped to the bottom, turned to 180 degrees
- moved C21 152.8 mm to (94.0, 14.0), flipped to the bottom, turned to 180 degrees
- moved C32 145.4 mm to (45.7, 2.54), flipped to the bottom
- moved R22 145.1 mm to (64.8, 20.3)
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Routing:
- net +3V3: track 29.1 -> 303.3 mm, vias 8 -> 21
- net MODE_SEL[1]: track 0.00 -> 58.6 mm, vias 0 -> 2
- net MODE_SEL[0]: track 0.00 -> 57.9 mm, vias 0 -> 2
- net DS4_GREEN/VID_SEL[0]: track 45.4 -> 99.6 mm, vias 1 -> 3
- net DS4_PWREN/CDP_EN: track 0.00 -> 54.0 mm, vias 0 -> 2
- net DS1_PWREN/CDP_EN: track 0.00 -> 51.9 mm, vias 0 -> 2
- net DS1_OVRCURR: track 0.00 -> 51.5 mm, vias 0 -> 2
- net PWR_SW_POL: track 0.00 -> 50.7 mm, vias 0 -> 2
- net +5V: track 0.63 -> 50.2 mm, vias 1 -> 9
- net DS4_OVRCURR: track 0.00 -> 47.3 mm, vias 0 -> 2
- net US_OVRCURR: track 0.00 -> 45.6 mm, vias 0 -> 2
- net DS2_GREEN/NON_REMOVABLE[1]: track 58.9 -> 93.5 mm
- net DS1_RX_N: track 67.5 -> 35.4 mm
- net RESETIN: track 72.4 -> 40.3 mm, vias 1 -> 2
- net DS1_D_P: track 90.4 -> 59.0 mm
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- added copper zone on layer 15, net +5V
Other:
- board size 101.6 x 50.8 mm -> 97.8 x 45.7 mm
- board text added: "Ethan Kessel"
- board text added: "HX3 CYUSB 3.0 HUB"
